File: hardware-HSSM-HVPCB/HSSM-HVPCB.kicad_sch (KiCad schematic)
At the start: 65 parts, among them J1 2601-1108, J3 Connector_BTB_20021311-00010T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, K1 G6DN-1A-L DC12, K2 G6DN-1A-L DC12, Q1 Q_NMOS_SOT-23_IRLML6344, Q2 Q_NMOS_SOT-23_IRLML6344, U1 LNK3204D-TL, U2 CS5480-INZ, U3 LTV-354T, U4 LTV-354T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

Commit message: [#7] Placement WIP
Parts:
- removed J1: 2601-1108, HSSM-HVPCB:2601-1108, symbol HSSM-HVPCB:terminal_1x8_2601-1108_wago
- added J2: 805-108, HSSM-HVPCB:805-108, symbol HSSM-HVPCB:Push-in_terminal-1x08_WAGO_805-108
Connections:
- net AC_L: now also J2.3, J2.5
- net AC_N: now also J2.6
- net AC_Q1: now also J2.8
- net AC_Q2: now also J2.1
- net AC_S1: now also J2.7
- net AC_S2: now also J2.2
- net AC_S3: now also J2.4
Changed lines of the file:
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@@
 	(wire
 		(pts
+			(xy 297.18 222.25) (xy 297.18 224.79)
+		)
+		(stroke
+			(width 0)
+			(type default)
+		)
+	)
+	(wire
+		(pts
 			(xy 133.35 233.68) (xy 142.24 233.68)
 		)
@@
 	(wire
 		(pts
-			(xy 297.18 224.79) (xy 297.18 222.25)
-		)
-		(stroke
-			(width 0)
-			(type default)
-		)
-	)
-	(wire
-		(pts
 			(xy 369.57 71.12) (xy 381 71.12)
 		)
@@
 	)
 	(symbol
+		(lib_id "power:AC")
+		(at 297.18 222.25 0)
+		(unit 1)
+		(exclude_from_sim no)
+		(in_bom yes)
+		(on_board yes)
+		(dnp no)
+		(property "Reference" "#PWR032"
+			(at 297.18 224.79 0)
+			(effects
+				(font
+					(size 1.27 1.27)
+				)
+				(hide yes)
+			)
+		)
+		(property "Value" "AC_L"
+			(at 297.18 214.122 90)
+			(effects
+				(font
+					(size 1.27 1.27)
+				)
+			)
+		)
+		(property "Footprint" ""
+			(at 297.18 222.25 0)
+			(effects
+				(font
+					(size 1.27 1.27)
+				)
+				(hide yes)
+			)
+		)
+		(property "Datasheet" ""
+			(at 297.18 222.25 0)
+			(effects
+				(font
+					(size 1.27 1.27)
+				)
+				(hide yes)
+			)
+		)
+		(property "Description" "Power symbol creates a global label with name \"AC\""
+			(at 297.18 222.25 0)
+			(effects
+				(font
+					(size 1.27 1.27)
+				)
+				(hide yes)
+			)
+		)
+		(pin "1"
+		)
+		(instances
+			(project "HSSM-HVPCB"
+				(path "/e1056638-7c6b-48e4-9e2e-c0f7b783eee5"
+					(reference "#PWR032")
+					(unit 1)
+				)
+			)
+		)
+	)
+	(symbol
 		(lib_id "power:GND")
 		(at 100.33 241.3 0)
@@
 	)
 	(symbol
-		(lib_id "power:AC")
-		(at 292.1 222.25 0)
-		(unit 1)
-		(exclude_from_sim no)
-		(in_bom yes)
-		(on_board yes)
-		(dnp no)
-		(property "Reference" "#PWR033"
-			(at 292.1 224.79 0)
-			(effects
-				(font
-					(size 1.27 1.27)
-				)
-				(hide yes)
-			)
-		)
-		(property "Value" "AC_L"
-			(at 292.1 214.122 90)
-			(effects
-				(font
-					(size 1.27 1.27)
-				)
-			)
-		)
-		(property "Footprint" ""
-			(at 292.1 222.25 0)
-			(effects
-				(font
-					(size 1.27 1.27)
-				)
-				(hide yes)
-			)
-		)
-		(property "Datasheet" ""
-			(at 292.1 222.25 0)
-			(effects
-				(font
-					(size 1.27 1.27)
-				)
-				(hide yes)
-			)
-		)
-		(property "Description" "Power symbol creates a global label with name \"AC\""
-			(at 292.1 222.25 0)
-			(effects
-				(font
-					(size 1.27 1.27)
-				)
-				(hide yes)
-			)
-		)
-		(pin "1"
-		)
-		(instances
-			(project "HSSM-HVPCB"
-				(path "/e1056638-7c6b-48e4-9e2e-c0f7b783eee5"
-					(reference "#PWR033")
-					(unit 1)
-				)
-			)
-		)
-	)
-	(symbol
 		(lib_id "power:GND")
 		(at 386.08 73.66 0)
@@
 	)
 	(symbol
-		(lib_id "HSSM-HVPCB:terminal_1x8_2601-1108_wago")
-		(at 289.56 234.95 90)
-		(mirror x)
+		(lib_id "power:AC")
+		(at 101.6 64.77 0)
 		(unit 1)
 		(exclude_from_sim no)
@@
 		(on_board yes)
 		(dnp no)
-		(property "Reference" "J1"
-			(at 289.56 238.76 90)
+		(property "Reference" "#PWR041"
+			(at 101.6 67.31 0)
 			(effects
 				(font
 					(size 1.27 1.27)
 				)
+				(hide yes)
 			)
 		)
-		(property "Value" "2601-1108"
-			(at 289.56 241.3 90)
+		(property "Value" "AC_L"
+			(at 101.6 58.166 0)
 			(effects
 				(font
@@
 			)
 		)
-		(property "Footprint" "HSSM-HVPCB:2601-1108"
-			(at 290.83 234.95 0)
+		(property "Footprint" ""
+			(at 101.6 64.77 0)
 			(effects
 				(font
@@
 			)
 		)
-		(property "Datasheet" "https://source.z2data.com/2022/11/30/3/26/12/266816/8679706/WAGO26011108enUS.pdf"
-			(at 290.83 234.95 0)
+		(property "Datasheet" ""
+			(at 101.6 64.77 0)
 			(effects
 				(font
@@
 			)
 		)
-		(property "Description" "terminal_1x10_2601-1108_wago"
-			(at 290.83 234.95 0)
+		(property "Description" "Power symbol creates a global label with name \"AC\""
+			(at 101.6 64.77 0)
 			(effects
 				(font
@@
 			)
 		)
-		(property "MPN" "2601-1108"
-			(at 289.56 243.84 90)
-			(effects
-				(font
-					(size 1.27 1.27)
-				)
-			)
-		)
-		(property "Manufacturer" "WAGO"
-			(at 289.56 246.38 90)
-			(effects
-				(font
-					(size 1.27 1.27)
-				)
-			)
-		)
-		(pin "3"
-		)
-		(pin "2"
-		)
 		(pin "1"
 		)
-		(pin "7"
-		)
-		(pin "4"
-		)
-		(pin "5"
-		)
-		(pin "6"
-		)
-		(pin "8"
-		)
 		(instances
-			(project ""
+			(project "HSSM-HVPCB"
 				(path "/e1056638-7c6b-48e4-9e2e-c0f7b783eee5"
-					(reference "J1")
+					(reference "#PWR041")
 					(unit 1)
 				)
@@
 	)
 	(symbol
-		(lib_id "power:AC")
-		(at 101.6 64.77 0)
+		(lib_id "power:+3V3")
+		(at 64.77 176.53 0)
 		(unit 1)
 		(exclude_from_sim no)
@@
 		(on_board yes)
 		(dnp no)
-		(property "Reference" "#PWR041"
-			(at 101.6 67.31 0)
+		(fields_autoplaced yes)
+		(property "Reference" "#PWR061"
+			(at 64.77 180.34 0)
 			(effects
 				(font
@@
 			)
 		)
-		(property "Value" "AC_L"
-			(at 101.6 58.166 0)
+		(property "Value" "+3V3"
+			(at 64.77 171.45 0)
 			(effects
 				(font
@@
 		)
 		(property "Footprint" ""
-			(at 101.6 64.77 0)
+			(at 64.77 176.53 0)
 			(effects
 				(font
@@
 		)
 		(property "Datasheet" ""
-			(at 101.6 64.77 0)
+			(at 64.77 176.53 0)
 			(effects
 				(font
@@
 			)
 		)
-		(property "Description" "Power symbol creates a global label with name \"AC\""
-			(at 101.6 64.77 0)
+		(property "Description" "Power symbol creates a global label with name \"+3V3\""
+			(at 64.77 176.53 0)
 			(effects
 				(font
@@
 			(project "HSSM-HVPCB"
 				(path "/e1056638-7c6b-48e4-9e2e-c0f7b783eee5"
-					(reference "#PWR041")
+					(reference "#PWR061")
 					(unit 1)
 				)
@@
 	)
 	(symbol
-		(lib_id "power:+3V3")
-		(at 64.77 176.53 0)
+		(lib_id "HSSM-HVPCB:Push-in_terminal-1x08_WAGO_805-108")
+		(at 298.45 229.87 270)
 		(unit 1)
 		(exclude_from_sim no)
@@
 		(dnp no)
 		(fields_autoplaced yes)
-		(property "Reference" "#PWR061"
-			(at 64.77 180.34 0)
+		(property "Reference" "J2"
+			(at 302.26 234.9499 90)
+			(effects
+				(font
+					(size 1.524 1.524)
+				)
+				(justify left)
+			)
+		)
+		(property "Value" "805-108"
+			(at 302.26 237.4899 90)
+			(effects
+				(font
+					(size 1.524 1.524)
+				)
+				(justify left)
+			)
+		)
+		(property "Footprint" "HSSM-HVPCB:805-108"
+			(at 298.45 229.87 0)
 			(effects
 				(font
 					(size 1.27 1.27)
+					(italic yes)
 				)
 				(hide yes)
 			)
 		)
-		(property "Value" "+3V3"
-			(at 64.77 171.45 0)
+		(property "Datasheet" "805-108"
+			(at 298.45 229.87 0)
 			(effects
 				(font
 					(size 1.27 1.27)
+					(italic yes)
 				)
+				(hide yes)
 			)
 		)
-		(property "Footprint" ""
-			(at 64.77 176.53 0)
+		(property "Description" ""
+			(at 298.45 229.87 0)
 			(effects
 				(font
@@
 			)
 		)
-		(property "Datasheet" ""
-			(at 64.77 176.53 0)
+		(property "Manufacturer" "WAGO"
+			(at 302.26 240.0299 90)
 			(effects
 				(font
 					(size 1.27 1.27)
 				)
-				(hide yes)
+				(justify left)
 			)
 		)
-		(property "Description" "Power symbol creates a global label with name \"+3V3\""
-			(at 64.77 176.53 0)
+		(property "MPN" "805-108"
+			(at 302.26 242.5699 90)
 			(effects
 				(font
 					(size 1.27 1.27)
 				)
-				(hide yes)
+				(justify left)
 			)
 		)
+		(pin "4"
+		)
+		(pin "3"
+		)
+		(pin "5"
+		)
+		(pin "6"
+		)
 		(pin "1"
 		)
+		(pin "2"
+		)
+		(pin "7"
+		)
+		(pin "8"
+		)
 		(instances
-			(project "HSSM-HVPCB"
+			(project ""
 				(path "/e1056638-7c6b-48e4-9e2e-c0f7b783eee5"
-					(reference "#PWR061")
+					(reference "J2")
 					(unit 1)
 				)
@@
 	(symbol
 		(lib_id "power:AC")
-		(at 297.18 222.25 0)
+		(at 292.1 222.25 0)
 		(unit 1)
 		(exclude_from_sim no)
@@
 		(dnp no)
 		(property "Reference" "#PWR034"
-			(at 297.18 224.79 0)
+			(at 292.1 224.79 0)
 			(effects
 				(font
@@
 		)
 		(property "Value" "AC_S3"
-			(at 297.18 213.868 90)
+			(at 292.1 213.868 90)
 			(effects
 				(font
@@
 		)
 		(property "Footprint" ""
-			(at 297.18 222.25 0)
+			(at 292.1 222.25 0)
 			(effects
 				(font
@@
 		)
 		(property "Datasheet" ""
-			(at 297.18 222.25 0)
+			(at 292.1 222.25 0)
 			(effects
 				(font
@@
 		)
 		(property "Description" "Power symbol creates a global label with name \"AC\""
-			(at 297.18 222.25 0)
+			(at 292.1 222.25 0)
 			(effects
 				(font

Commit message: [#7] Placement WIP
Parts:
- added CON1: ~, HSSM-HVPCB:FFC_solder_connector_16pos, symbol HSSM-HVPCB:FFC_solder_connector_16pos
- added R9: R_10_5pct_Axial_RR02J10RTB, HSSM-HVPCB:R_Axial_DIN0204_L3.6mm_D1.6mm_P2.54mm_Vertical, symbol HSSM-HVPCB:R_10_5pct_Axial_RR02J10RTB
Connections:
- net AC_N: now also R9.1; no longer D2.2 (A)
- new net: D2.2 (A), R9.2
Changed lines of the file:
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@@
 	(wire
 		(pts
-			(xy 269.24 59.69) (xy 262.89 59.69)
-		)
-		(stroke
-			(width 0)
-			(type default)
-		)
-	)
-	(wire
-		(pts
 			(xy 110.49 241.3) (xy 115.57 241.3)
 		)
@@
 	(wire
 		(pts
+			(xy 265.43 59.69) (xy 269.24 59.69)
+		)
+		(stroke
+			(width 0)
+			(type default)
+		)
+	)
+	(wire
+		(pts
 			(xy 369.57 36.83) (xy 369.57 40.64)
 		)
@@
 	(wire
 		(pts
+			(xy 256.54 59.69) (xy 260.35 59.69)
+		)
+		(stroke
+			(width 0)
+			(type default)
+		)
+	)
+	(wire
+		(pts
 			(xy 124.46 100.33) (xy 134.62 100.33)
 		)
@@
 	)
 	(symbol
+		(lib_id "HSSM-HVPCB:FFC_solder_connector_16pos")
+		(at 158.75 184.15 90)
+		(unit 1)
+		(exclude_from_sim no)
+		(in_bom no)
+		(on_board yes)
+		(dnp no)
+		(fields_autoplaced yes)
+		(property "Reference" "CON1"
+			(at 158.75 172.72 90)
+			(effects
+				(font
+					(size 1.27 1.27)
+				)
+			)
+		)
+		(property "Value" "~"
+			(at 158.75 175.26 90)
+			(effects
+				(font
+					(size 1.27 1.27)
+				)
+			)
+		)
+		(property "Footprint" "HSSM-HVPCB:FFC_solder_connector_16pos"
+			(at 153.67 184.15 0)
+			(effects
+				(font
+					(size 1.27 1.27)
+				)
+				(hide yes)
+			)
+		)
+		(property "Datasheet" ""
+			(at 153.67 184.15 0)
+			(effects
+				(font
+					(size 1.27 1.27)
+				)
+				(hide yes)
+			)
+		)
+		(property "Description" ""
+			(at 153.67 184.15 0)
+			(effects
+				(font
+					(size 1.27 1.27)
+				)
+				(hide yes)
+			)
+		)
+		(pin "1"
+		)
+		(pin "6"
+		)
+		(pin "14"
+		)
+		(pin "8"
+		)
+		(pin "7"
+		)
+		(pin "9"
+		)
+		(pin "12"
+		)
+		(pin "10"
+		)
+		(pin "11"
+		)
+		(pin "4"
+		)
+		(pin "13"
+		)
+		(pin "5"
+		)
+		(pin "16"
+		)
+		(pin "2"
+		)
+		(pin "15"
+		)
+		(pin "3"
+		)
+		(instances
+			(project ""
+				(path "/e1056638-7c6b-48e4-9e2e-c0f7b783eee5"
+					(reference "CON1")
+					(unit 1)
+				)
+			)
+		)
+	)
+	(symbol
 		(lib_id "HSSM-HVPCB:R_3k3_5pct_0402_RC0402JR-073K3L")
 		(at 381 60.96 90)
@@
 		(on_board yes)
 		(dnp no)
-		(fields_autoplaced yes)
 		(property "Reference" "#PWR021"
 			(at 295.91 125.73 0)
@@
 	)
 	(symbol
+		(lib_id "HSSM-HVPCB:R_10_5pct_Axial_RR02J10RTB")
+		(at 262.89 59.69 0)
+		(unit 1)
+		(exclude_from_sim no)
+		(in_bom yes)
+		(on_board yes)
+		(dnp no)
+		(fields_autoplaced yes)
+		(property "Reference" "R9"
+			(at 262.89 53.34 0)
+			(effects
+				(font
+					(size 1.27 1.27)
+					(thickness 0.15)
+				)
+			)
+		)
+		(property "Value" "R_10_5pct_Axial_RR02J10RTB"
+			(at 262.89 67.564 0)
+			(effects
+				(font
+					(size 1.27 1.27)
+					(thickness 0.15)
+				)
+				(justify left bottom)
+				(hide yes)
+			)
+		)
+		(property "Footprint" "HSSM-HVPCB:R_Axial_DIN0204_L3.6mm_D1.6mm_P2.54mm_Vertical"
+			(at 262.89 70.104 0)
+			(effects
+				(font
+					(size 1.27 1.27)
+					(thickness 0.15)
+				)
+				(justify left bottom)
+				(hide yes)
+			)
+		)
+		(property "Datasheet" "https://www.te.com/usa-en/product-3-1879352-7.datasheet.pdf"
+			(at 262.89 72.644 0)
+			(effects
+				(font
+					(size 1.27 1.27)
+					(thickness 0.15)
+				)
+				(justify left bottom)
+				(hide yes)
+			)
+		)
+		(property "Description" "SMD Resistor, 10Ω, ±5%, 0402, RR02J10RTB"
+			(at 262.89 59.69 0)
+			(effects
+				(font
+					(size 1.27 1.27)
+				)
+				(hide yes)
+			)
+		)
+		(property "MPN" "RR02J10RTB"
+			(at 262.89 75.184 0)
+			(effects
+				(font
+					(size 1.27 1.27)
+					(thickness 0.15)
+				)
+				(justify left bottom)
+				(hide yes)
+			)
+		)
+		(property "Manufacturer" "TE Connectivity"
+			(at 262.89 77.724 0)
+			(effects
+				(font
+					(size 1.27 1.27)
+					(thickness 0.15)
+				)
+				(justify left bottom)
+				(hide yes)
+			)
+		)
+		(property "License" "Apache-2.0"
+			(at 262.89 80.264 0)
+			(effects
+				(font
+					(size 1.27 1.27)
+				)
+				(justify left bottom)
+				(hide yes)
+			)
+		)
+		(property "Author" "Lukasz Nowarkiewicz"
+			(at 262.89 82.804 0)
+			(effects
+				(font
+					(size 1.27 1.27)
+				)
+				(justify left bottom)
+				(hide yes)
+			)
+		)
+		(property "Val" "10"
+			(at 262.89 55.88 0)
+			(effects
+				(font
+					(size 1.27 1.27)
+				)
+			)
+		)
+		(pin "1"
+		)
+		(pin "2"
+		)
+		(instances
+			(project ""
+				(path "/e1056638-7c6b-48e4-9e2e-c0f7b783eee5"
+					(reference "R9")
+					(unit 1)
+				)
+			)
+		)
+	)
+	(symbol
 		(lib_id "HSSM-HVPCB:R_499k_1pct_1206_KTR18EZPF4993")
 		(at 101.6 93.98 90)
@@
 	(symbol
 		(lib_id "power:AC")
-		(at 262.89 59.69 90)
+		(at 256.54 59.69 90)
 		(unit 1)
 		(exclude_from_sim no)
@@
 		(fields_autoplaced yes)
 		(property "Reference" "#PWR074"
-			(at 265.43 59.69 0)
+			(at 259.08 59.69 0)
 			(effects
 				(font
@@
 		)
 		(property "Value" "AC_N"
-			(at 256.54 59.6899 90)
+			(at 250.19 59.6899 90)
 			(effects
 				(font
@@
 		)
 		(property "Footprint" ""
-			(at 262.89 59.69 0)
+			(at 256.54 59.69 0)
 			(effects
 				(font
@@
 		)
 		(property "Datasheet" ""
-			(at 262.89 59.69 0)
+			(at 256.54 59.69 0)
 			(effects
 				(font
@@
 		)
 		(property "Description" "Power symbol creates a global label with name \"AC\""
-			(at 262.89 59.69 0)
+			(at 256.54 59.69 0)
 			(effects
 				(font
