File: hardware-HSSM-LVPCB/HSSM-LVPCB.kicad_pcb (KiCad board)
At the start: 4 copper layers, 36 x 12 mm, 57 parts, among them J1 UFL_R_SMT_1_10, J2 LPPB061NGCN-RC, Q1 Q_MOSFET_N_BSS123, Q2 Q_MOSFET_N_BSS123, U1 ESP32-C6, U2 W25Q64JVSSIQ_SOIC-8, X1 X_40MHz_SMD_ECS-2520SMV-400-F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

Commit message: [#13] PCB routing WIP flash
Parts:
- turned L2 to 90 degrees
- turned R5 to 180 degrees
Connections:
- C18 pad 2: /GPIO22 -> /S2_sym
- R16 pad 1: /GPIO22 -> /S2_sym
- S2 pad 1: /GPIO22 -> /S2_sym
- S2 pad 3: /GPIO22 -> /S2_sym
- U1 pad 33: /GPIO20 -> unconnected-(U1-SDIO_DATA0-Pad33)
- U1 pad 6: /GPIO0 -> unconnected-(U1-XTAL_32K_P-Pad6)
- U1 pad 7: /GPIO1 -> unconnected-(U1-XTAL_32K_N-Pad7)
- U1 pad 8: /GPIO2 -> unconnected-(U1-GPIO2-Pad8)
- U1 pad 9: unconnected-(U1-GPIO3-Pad9) -> /S2_sym
Routing:
- net Net-(U1-SPID): track 0.95 -> 23.3 mm, vias 1 -> 2
- net /GPIO23: track 3.51 -> 25.8 mm
- net Net-(U1-SPIQ): track 4.74 -> 26.0 mm
- net /SPID: track 21.4 -> 1.72 mm, vias 1 -> 0
- net /GPIO22: track 9.70 -> 0.00 mm, vias 2 -> 0
- net /S2_sym: track 0.00 -> 8.41 mm, vias 0 -> 1
- net unconnected-(U1-XTAL_32K_P-Pad6): track 0.00 -> 7.91 mm, vias 0 -> 1
- net /GPIO0: track 9.88 -> 16.1 mm, vias 2 -> 1
- net /GPIO_Q2: track 10.6 -> 15.8 mm
- net /GPIO2: track 3.20 -> 7.78 mm, vias 2 -> 1
- net /GPIO21: track 22.8 -> 25.6 mm
- net unconnected-(U1-GPIO2-Pad8): track 0.00 -> 2.56 mm, vias 0 -> 1
- net /SPICS0: track 27.2 -> 29.7 mm
- net VDD_SPI: track 50.2 -> 51.5 mm
- net Net-(U1-SPIWP): track 15.5 -> 16.0 mm

Commit message: [#13] PCB routing WIP RGB
Parts:
- moved R8 0.85 mm to (124.9, 122.9)
Connections:
- R11 pad 1: /GPIO1 -> /RGB_G
- R12 pad 1: /GPIO2 -> /RGB_R
- R13 pad 1: /GPIO0 -> /RGB_B
- U1 pad 10: unconnected-(U1-MTMS-Pad10) -> /LP_UART_RXD
- U1 pad 11: unconnected-(U1-MTDI-Pad11) -> /LP_UART_TXD
- U1 pad 18: /GPIO_S3 -> unconnected-(U1-GPIO12-Pad18)
- U1 pad 33: unconnected-(U1-SDIO_DATA0-Pad33) -> /RGB_B
- U1 pad 34: /GPIO21 -> /RGB_G
- U1 pad 35: /GPIO22 -> /RGB_R
- U1 pad 36: /GPIO23 -> unconnected-(U1-SDIO_DATA3-Pad36)
Routing:
- net /RGB_B: track 0.00 -> 40.2 mm
- net /RGB_R: track 0.00 -> 35.1 mm
- net /GPIO1: track 28.5 -> 0.00 mm, vias 2 -> 0
- net unconnected-(U1-XTAL_32K_N-Pad7): track 0.00 -> 27.8 mm, vias 0 -> 1
- net /RGB_G: track 0.00 -> 26.9 mm
- net /GPIO0: track 16.1 -> 0.00 mm, vias 1 -> 0
- net /GPIO2: track 7.78 -> 0.00 mm, vias 1 -> 0
- net VDD_SPI: track 51.5 -> 45.4 mm
- net /GPIO3: track 11.1 -> 16.4 mm, vias 1 -> 0
- net Net-(U1-SPIQ): track 26.0 -> 23.0 mm
- net /SPICS0: track 29.7 -> 27.2 mm
- net unconnected-(U1-GPIO12-Pad18): track 0.00 -> 1.80 mm, vias 0 -> 1
- net /GPIO_S3: track 4.30 -> 2.50 mm, vias 2 -> 1
- net /GPIO21: track 25.6 -> 24.9 mm

Commit message: [#13] PCB routing WIP RGB
Parts:
- moved C12 0.30 mm to (140.1, 120.8)
Connections:
- C17 pad 2: /GPIO21 -> /S1_sym
- R15 pad 1: /GPIO21 -> /S1_sym
- S1 pad 1: /GPIO21 -> /S1_sym
- S1 pad 3: /GPIO21 -> /S1_sym
- U1 pad 36: unconnected-(U1-SDIO_DATA3-Pad36) -> /S1_sym
Routing:
- net /S1_sym: track 0.00 -> 41.3 mm, vias 0 -> 1
- net /GPIO21: track 24.9 -> 0.00 mm, vias 2 -> 0
- net unconnected-(U1-XTAL_32K_N-Pad7): track 27.8 -> 3.98 mm
- net /RGB_B: track 40.2 -> 25.8 mm
- net /GPIO23: track 25.8 -> 12.3 mm, vias 2 -> 0
- net /RGB_R: track 35.1 -> 27.4 mm
- net /SPICS0: track 27.2 -> 29.2 mm
- net VDD_SPI: track 45.4 -> 46.2 mm
- net +3V3: track 12.6 -> 13.2 mm, vias 8 -> 7

Commit message: [#13] PCB routing WIP GPIO
Parts:
- moved S3 0.22 mm to (142.1, 114.4)
- moved S2 0.15 mm to (150.6, 114.3)
Connections:
- C16 pad 2: /GPIO3 -> /S_set
- R14 pad 1: /GPIO3 -> /S_set
- SW_USER1 pad 1: /GPIO3 -> /S_set
- SW_USER1 pad 3: /GPIO3 -> /S_set
- U1 pad 7: unconnected-(U1-XTAL_32K_N-Pad7) -> /S2_sym
- U1 pad 9: /S2_sym -> unconnected-(U1-GPIO3-Pad9)
Routing:
- net /LP_UART_RXD: track 0.00 -> 12.1 mm, vias 0 -> 1
- net /LP_UART_TXD: track 0.00 -> 12.0 mm, vias 0 -> 1
- net /GPIO23: track 12.3 -> 1.28 mm
- net /GPIO_Q2: track 15.8 -> 24.2 mm
- net unconnected-(U1-XTAL_32K_P-Pad6): track 7.91 -> 1.01 mm
- net unconnected-(U1-XTAL_32K_N-Pad7): track 3.98 -> 0.00 mm, vias 1 -> 0
- net /BOOT: track 16.7 -> 13.2 mm
- net /GPIO_S2: track 4.26 -> 7.37 mm
- net /S2_sym: track 8.41 -> 10.6 mm, vias 1 -> 2
- net unconnected-(U1-GPIO3-Pad9): track 0.00 -> 1.55 mm
- net unconnected-(U1-GPIO2-Pad8): track 2.56 -> 3.19 mm, vias 1 -> 0
- net unconnected-(U1-GPIO12-Pad18): track 1.80 -> 1.27 mm

Commit message: [#13] PCB routing WIP GPIO
Connections:
- C19 pad 2: /GPIO23 -> /S3_sym
- R17 pad 1: /GPIO23 -> /S3_sym
- S3 pad 1: /GPIO23 -> /S3_sym
- S3 pad 3: /GPIO23 -> /S3_sym
- U1 pad 16: /GPIO_Q2 -> unconnected-(U1-GPIO10-Pad16)
- U1 pad 19: /GPIO3 -> /S_set
- U1 pad 6: unconnected-(U1-XTAL_32K_P-Pad6) -> /GPIO_Q2
- U1 pad 8: unconnected-(U1-GPIO2-Pad8) -> /S3_sym
Routing:
- net /S3_sym: track 0.00 -> 18.9 mm, vias 0 -> 2
- net /GPIO3: track 16.3 -> 0.00 mm
- net /S_set: track 0.00 -> 16.3 mm
- net /GPIO_Q2: track 24.2 -> 20.9 mm
- net unconnected-(U1-GPIO2-Pad8): track 3.19 -> 0.00 mm
- net /S2_sym: track 10.6 -> 13.4 mm
- net unconnected-(U1-GPIO10-Pad16): track 0.00 -> 1.68 mm, vias 0 -> 1
- net /GPIO23: track 1.28 -> 0.00 mm
- net unconnected-(U1-XTAL_32K_P-Pad6): track 1.01 -> 0.00 mm, vias 1 -> 0

Commit message: [#13] PCB routing WIP flash
Parts:
- moved C12 3.02 mm to (142.9, 121.8), turned to 180 degrees
Routing:
- net /GPIO_Q1: track 27.5 -> 24.6 mm
- net Net-(U1-SPICLK): track 29.7 -> 26.7 mm
- net Net-(U1-SPIHD): track 32.2 -> 30.1 mm
- net Net-(U1-SPIWP): track 16.0 -> 14.1 mm
- net GND: track 43.2 -> 44.4 mm
- net Net-(U1-SPID): track 23.3 -> 24.2 mm
- net /RGB_B: track 25.8 -> 25.0 mm
- net /RGB_G: track 26.4 -> 25.7 mm
- net /RGB_R: track 27.4 -> 26.6 mm
- net +3V3: track 13.2 -> 12.5 mm, vias 7 -> 8

Commit message: [#13] PCB routing WIP flash
Routing:
- net VDD_SPI: track 46.2 -> 33.0 mm, vias 3 -> 2
- net Net-(U1-SPIQ): track 23.1 -> 19.5 mm
- net /SPICS0: track 29.2 -> 30.9 mm, vias 2 -> 4

Commit message: [#13] PCB routing WIP GPIO
Parts:
- moved R2 0.67 mm to (129.8, 118.2), turned to -90 degrees
- moved R1 0.05 mm to (129.8, 120.5)
Routing:
- net /DO1: track 2.20 -> 30.4 mm
- net /GPIO_S3: track 2.15 -> 28.8 mm, vias 1 -> 2
- net /GPIO_S2: track 7.37 -> 29.5 mm, vias 2 -> 3
- net /GPIO_Q2: track 20.9 -> 40.6 mm, vias 3 -> 4
- net /BOOT: track 13.2 -> 2.46 mm
- net +12V: track 0.00 -> 1.95 mm, vias 0 -> 1
- net GND: track 44.4 -> 46.3 mm, vias 21 -> 22
- net /LP_UART_TXD: track 12.0 -> 13.4 mm
- net +3V3: track 12.5 -> 13.2 mm, vias 8 -> 9
- net Net-(U1-SPIWP): track 14.1 -> 14.7 mm
