File: hardware-HSSM-FCB/HSSM-FCB.kicad_sch (KiCad schematic)
At the start: 2 parts

Commit message: HSSM-FCB add fabrication files
Other:
- title: (none) -> HSSM-FCB
Changed lines of the file:
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@@
 	(generator_version "8.0")
 	(paper "A4")
+	(title_block
+		(title "HSSM-FCB")
+		(date "2025-01-22")
+		(rev "1.0.0")
+	)
 	(wire
 		(pts
